Commit message: joint_state_publisher gui looks working

File: sample_diff_drive_description/urdf/vehicle.xacro (robot description, xacro)
@@ -29,7 +29,9 @@
   <!-- left wheel -->
   <joint name="left_wheel_joint" type="continuous">
+	<!-- if axis tag is not specified for continuous, the joint/link flickers -->
+	<axis xyz="0 1 0"/>
+	<origin xyz="0 -${vehicle_width/2.0} 0" rpy="0 0 0"/>
 	<parent link="base_link"/>
 	<child link="left_wheel_link"/>
-	<origin xyz="0 -${vehicle_width/2.0} 0" rpy="0 0 0"/>
   </joint>
   <link name="left_wheel_link">
@@ -43,7 +45,9 @@
   <!-- right wheel -->
   <joint name="right_wheel_joint" type="continuous">
+	<!-- if axis tag is not specified for continuous, the joint/link flickers -->
+	<axis xyz="0 1 0"/>
+	<origin xyz="0 ${vehicle_width/2.0} 0" rpy="0 0 0"/>
 	<parent link="base_link"/>
 	<child link="right_wheel_link"/>
-	<origin xyz="0 ${vehicle_width/2.0} 0" rpy="0 0 0"/>
   </joint>
   <link name="right_wheel_link">

Commit message: adding color, will fix dirction

File: sample_diff_drive_description/urdf/vehicle.xacro (robot description, xacro)
@@ -24,4 +24,7 @@
 		<box size="${vehicle_length} ${vehicle_width} ${vehicle_height}"/>
 	  </geometry>
+	  <material name="gray">
+		<color rgba="1.0 1.0 1.0 0.8"/>
+	  </material>
 	</visual>
   </link>
@@ -41,4 +44,7 @@
 		<cylinder radius="${wheel_radius}" length="${wheel_width}"/>
 	  </geometry>
+	  <material name="red">
+		<color rgba="1.0 0.0 0.0 0.8"/>
+	  </material>
 	</visual>
   </link>
@@ -57,6 +63,25 @@
 		<cylinder radius="${wheel_radius}" length="${wheel_width}"/>
 	  </geometry>
+	  <material name="red">
+		<color rgba="1.0 0.0 0.0 0.8"/>
+	  </material>
 	</visual>
   </link>
   <!-- front caster -->
+  <joint name="caster_joint" type="fixed">
+	<parent link="base_link"/>
+	<child link="caster_wheel"/>
+	<origin xyz="${front_overhang * 0.9} 0 0" rpy="0 0 0"/>
+  </joint>
+  <link name="caster_wheel">
+	<visual>
+	  <origin xyz="0 0 0" rpy="${pi/2} 0 0"/>
+	  <geometry>
+		<cylinder radius="${wheel_radius}" length="${wheel_width}"/>
+	  </geometry>
+	  <material name="white">
+		<color rgba="1.0 1.0 1.0 0.8"/>
+	  </material>
+	</visual>
+  </link>
 </robot>

Commit message: need to add offset of wheel to the ground

File: sample_diff_drive_description/urdf/vehicle.xacro (robot description, xacro)
@@ -15,6 +15,5 @@
 	<parent link="base_link"/>
 	<child link="vehicle_body"/>
-	<origin xyz="${vehicle_length/2.0 - rear_overhang} 0 ${wheel_radius}"
-			rpy="0 0 0"/>
+	<origin xyz="${vehicle_length/2 - rear_overhang} 0 ${wheel_radius}" rpy="0 0 0"/>
   </joint>
   <link name="vehicle_body">

Commit message: added base_footprint

File: sample_diff_drive_description/urdf/vehicle.xacro (robot description, xacro)
@@ -9,4 +9,11 @@
   <xacro:property name="vehicle_length" value="${vehicle_info['/**']['ros__parameters']['vehicle_length']}"/>
   <xacro:property name="vehicle_height" value="${vehicle_info['/**']['ros__parameters']['vehicle_height']}"/>
+  <!-- coordinate (x, y, 0) -->
+  <link name="base_footprint"/>
+  <joint name="virtual_footprint_joint" type="fixed">
+	<parent link="base_footprint"/>
+	<child link="base_link"/>
+	<origin xyz="0 0 ${wheel_radius}" rpy="0 0 0"/>
+  </joint>
   <!-- the center of wheels (for control/planning) -->
   <link name="base_link"/>

Commit message: changed caster wheel size. Looks good

File: sample_diff_drive_description/urdf/vehicle.xacro (robot description, xacro)
@@ -9,4 +9,5 @@
   <xacro:property name="vehicle_length" value="${vehicle_info['/**']['ros__parameters']['vehicle_length']}"/>
   <xacro:property name="vehicle_height" value="${vehicle_info['/**']['ros__parameters']['vehicle_height']}"/>
+  <xacro:property name="caster_wheel_radius" value="${vehicle_info['/**']['ros__parameters']['caster_wheel_radius']}"/>
   <!-- coordinate (x, y, 0) -->
   <link name="base_footprint"/>
@@ -76,7 +77,7 @@
   <!-- front caster -->
   <joint name="caster_joint" type="fixed">
-	<parent link="base_link"/>
+	<parent link="base_footprint"/>
 	<child link="caster_wheel"/>
-	<origin xyz="${front_overhang * 0.9} 0 0" rpy="0 0 0"/>
+	<origin xyz="${front_overhang * 0.9} 0 ${caster_wheel_radius}" rpy="0 0 0"/>
   </joint>
   <link name="caster_wheel">
@@ -84,5 +85,5 @@
 	  <origin xyz="0 0 0" rpy="${pi/2} 0 0"/>
 	  <geometry>
-		<cylinder radius="${wheel_radius}" length="${wheel_width}"/>
+		<cylinder radius="${caster_wheel_radius}" length="${wheel_width}"/>
 	  </geometry>
 	  <material name="white">

Commit message: disabled continuous joint of two wheels

File: sample_diff_drive_description/urdf/vehicle.xacro (robot description, xacro)
@@ -38,7 +38,5 @@
   <!-- two wheels -->
   <!-- left wheel -->
-  <joint name="left_wheel_joint" type="continuous">
-	<!-- if axis tag is not specified for continuous, the joint/link flickers -->
-	<axis xyz="0 1 0"/>
+  <joint name="left_wheel_joint" type="fixed">
 	<origin xyz="0 -${vehicle_width/2.0} 0" rpy="0 0 0"/>
 	<parent link="base_link"/>
@@ -57,7 +55,6 @@
   </link>
   <!-- right wheel -->
-  <joint name="right_wheel_joint" type="continuous">
+  <joint name="right_wheel_joint" type="fixed">
 	<!-- if axis tag is not specified for continuous, the joint/link flickers -->
-	<axis xyz="0 1 0"/>
 	<origin xyz="0 ${vehicle_width/2.0} 0" rpy="0 0 0"/>
 	<parent link="base_link"/>
